Commit message: Add URDF link name

File: urdf/atom.urdf (robot description, URDF)
Before this commit: robot atom, 31 links, 30 joints
Links:
- removed link uidx_arm_l1_link
- removed link uidx_arm_l2_link
- removed link uidx_arm_r1_link
- removed link uidx_arm_r2_link
- added link left_elbow_pitch_link, mass 0.8548; collision box size=0.30 0.06 0.06; visual mesh filename=package://atom_urdf/meshes/left_elbow_pitch_link.STL
- added link left_shoulder_pitch_link, mass 0.4473; visual mesh filename=package://atom_urdf/meshes/left_shoulder_pitch_link.STL
- added link right_elbow_pitch_link, mass 0.8548; collision box size=0.30 0.06 0.06; visual mesh filename=package://atom_urdf/meshes/right_elbow_pitch_link.STL
- added link right_shoulder_pitch_link, mass 0.4473; visual mesh filename=package://atom_urdf/meshes/right_shoulder_pitch_link.STL
- link head_pitch_link: geometry collision box size=0.16 0.14 0.14; visual mesh filename=package://atom_urdf/meshes/head_pitch_link.STL
- link head_yaw_link: geometry visual mesh filename=package://atom_urdf/meshes/head_yaw_link.STL
- link left_elbow_roll_link: geometry visual mesh filename=package://atom_urdf/meshes/left_elbow_roll_link.STL
- link left_shoulder_roll_link: geometry collision box size=0.06 0.06 0.24; visual mesh filename=package://atom_urdf/meshes/left_shoulder_roll_link.STL
- link left_shoulder_yaw_link: geometry visual mesh filename=package://atom_urdf/meshes/left_shoulder_yaw_link.STL
- link left_wrist_pitch_link: geometry visual mesh filename=package://atom_urdf/meshes/left_wrist_pitch_link.STL
- link left_wrist_yaw_link: geometry visual mesh filename=package://atom_urdf/meshes/left_wrist_yaw_link.STL
- link leg_l1_link: geometry visual mesh filename=package://atom_urdf/meshes/leg_l1_link.STL
- link leg_l2_link: geometry visual mesh filename=package://atom_urdf/meshes/leg_l2_link.STL
- link leg_l3_link: geometry collision box size=0.08 0.08 0.24; visual mesh filename=package://atom_urdf/meshes/leg_l3_link.STL
- link leg_l4_link: geometry collision box size=0.08 0.08 0.32; visual mesh filename=package://atom_urdf/meshes/leg_l4_link.STL
- link leg_l5_link: geometry visual mesh filename=package://atom_urdf/meshes/leg_l5_link.STL
- link leg_l6_link: geometry collision box size=0.25 0.1 0.02; visual mesh filename=package://atom_urdf/meshes/leg_l6_link.STL
- link leg_r1_link: geometry visual mesh filename=package://atom_urdf/meshes/leg_r1_link.STL
- link leg_r2_link: geometry visual mesh filename=package://atom_urdf/meshes/leg_r2_link.STL
- link leg_r3_link: geometry collision box size=0.08 0.08 0.24; visual mesh filename=package://atom_urdf/meshes/leg_r3_link.STL
- link leg_r4_link: geometry collision box size=0.08 0.08 0.32; visual mesh filename=package://atom_urdf/meshes/leg_r4_link.STL
- link leg_r5_link: geometry visual mesh filename=package://atom_urdf/meshes/leg_r5_link.STL
- link leg_r6_link: geometry collision box size=0.25 0.1 0.02; visual mesh filename=package://atom_urdf/meshes/leg_r6_link.STL
- link pelvis: geometry visual mesh filename=package://atom_urdf/meshes/pelvis.STL
- link right_elbow_roll_link: geometry visual mesh filename=package://atom_urdf/meshes/right_elbow_roll_link.STL
- link right_shoulder_roll_link: geometry collision box size=0.06 0.06 0.24; visual mesh filename=package://atom_urdf/meshes/right_shoulder_roll_link.STL
- link right_shoulder_yaw_link: geometry visual mesh filename=package://atom_urdf/meshes/right_shoulder_yaw_link.STL
- link right_wrist_pitch_link: geometry visual mesh filename=package://atom_urdf/meshes/right_wrist_pitch_link.STL
- link right_wrist_yaw_link: geometry visual mesh filename=package://atom_urdf/meshes/right_wrist_yaw_link.STL
- link torso_link: geometry collision box size=0.26 0.24 0.4; visual mesh filename=package://atom_urdf/meshes/torso_link.STL
Joints:
- removed joint uidx_l_arm_joint1
- removed joint uidx_l_arm_joint2
- removed joint uidx_r_arm_joint1
- removed joint uidx_r_arm_joint2
- added joint left_elbow_pitch_joint: type revolute, parent left_shoulder_yaw_link, child left_elbow_pitch_link, origin xyz=0.00044198773719138 0 -0.130000000000198 rpy=0 0 0, axis 0 1 0, limit lower=-1.57 upper=2 effort=36 velocity=2.62
- added joint left_shoulder_pitch_joint: type revolute, parent torso_link, child left_shoulder_pitch_link, origin xyz=0 0.128 0.333 rpy=0 0 0, axis 0 1 0, limit lower=-2.97 upper=2.97 effort=56 velocity=2.62
- added joint right_elbow_pitch_joint: type revolute, parent right_shoulder_yaw_link, child right_elbow_pitch_link, origin xyz=0.000441987737191488 0 -0.130000000000198 rpy=0 0 0, axis 0 1 0, limit lower=-1.57 upper=2 effort=36 velocity=2.62
- added joint right_shoulder_pitch_joint: type revolute, parent torso_link, child right_shoulder_pitch_link, origin xyz=0 -0.128 0.333 rpy=0 0 0, axis 0 1 0, limit lower=-2.97 upper=2.97 effort=56 velocity=2.62
- joint head_pitch_joint: type fixed -> revolute
- joint head_yaw_joint: type fixed -> revolute
- joint left_elbow_roll_joint: parent uidx_arm_l2_link -> left_elbow_pitch_link; type fixed -> revolute
- joint left_shoulder_roll_joint: parent uidx_arm_l1_link -> left_shoulder_pitch_link; type fixed -> revolute
- joint left_shoulder_yaw_joint: type fixed -> revolute
- joint left_wrist_pitch_joint: type fixed -> revolute
- joint left_wrist_yaw_joint: type fixed -> revolute
- joint right_elbow_roll_joint: parent uidx_arm_r2_link -> right_elbow_pitch_link; type fixed -> revolute
- joint right_shoulder_roll_joint: parent uidx_arm_r1_link -> right_shoulder_pitch_link; type fixed -> revolute
- joint right_shoulder_yaw_joint: type fixed -> revolute
- joint right_wrist_pitch_joint: type fixed -> revolute
- joint right_wrist_yaw_joint: type fixed -> revolute
- joint torso_joint: type fixed -> revolute

File: urdf/atom_lower.urdf (robot description, URDF)
Before this commit: robot atom, 32 links, 31 joints
Links:
- removed link uidx_arm_l1_link
- removed link uidx_arm_l2_link
- removed link uidx_arm_r1_link
- removed link uidx_arm_r2_link
- added link left_elbow_pitch_link, mass 0.8548; collision box size=0.30 0.06 0.06; visual mesh filename=package://atom_urdf/meshes/left_elbow_pitch_link.STL
- added link left_shoulder_pitch_link, mass 0.4473; visual mesh filename=package://atom_urdf/meshes/left_shoulder_pitch_link.STL
- added link right_elbow_pitch_link, mass 0.8548; collision box size=0.30 0.06 0.06; visual mesh filename=package://atom_urdf/meshes/right_elbow_pitch_link.STL
- added link right_shoulder_pitch_link, mass 0.4473; visual mesh filename=package://atom_urdf/meshes/right_shoulder_pitch_link.STL
- link head_pitch_link: geometry collision box size=0.16 0.14 0.14; visual mesh filename=package://atom_urdf/meshes/head_pitch_link.STL
- link head_yaw_link: geometry visual mesh filename=package://atom_urdf/meshes/head_yaw_link.STL
- link left_elbow_roll_link: geometry visual mesh filename=package://atom_urdf/meshes/left_elbow_roll_link.STL
- link left_shoulder_roll_link: geometry collision box size=0.06 0.06 0.24; visual mesh filename=package://atom_urdf/meshes/left_shoulder_roll_link.STL
- link left_shoulder_yaw_link: geometry visual mesh filename=package://atom_urdf/meshes/left_shoulder_yaw_link.STL
- link left_wrist_pitch_link: geometry visual mesh filename=package://atom_urdf/meshes/left_wrist_pitch_link.STL
- link left_wrist_yaw_link: geometry visual mesh filename=package://atom_urdf/meshes/left_wrist_yaw_link.STL
- link leg_l1_link: geometry visual mesh filename=package://atom_urdf/meshes/leg_l1_link.STL
- link leg_l2_link: geometry visual mesh filename=package://atom_urdf/meshes/leg_l2_link.STL
- link leg_l3_link: geometry collision box size=0.08 0.08 0.24; visual mesh filename=package://atom_urdf/meshes/leg_l3_link.STL
- link leg_l4_link: geometry collision box size=0.08 0.08 0.32; visual mesh filename=package://atom_urdf/meshes/leg_l4_link.STL
- link leg_l5_link: geometry visual mesh filename=package://atom_urdf/meshes/leg_l5_link.STL
- link leg_l6_link: geometry collision box size=0.25 0.1 0.02; visual mesh filename=package://atom_urdf/meshes/leg_l6_link.STL
- link leg_r1_link: geometry visual mesh filename=package://atom_urdf/meshes/leg_r1_link.STL
- link leg_r2_link: geometry visual mesh filename=package://atom_urdf/meshes/leg_r2_link.STL
- link leg_r3_link: geometry collision box size=0.08 0.08 0.24; visual mesh filename=package://atom_urdf/meshes/leg_r3_link.STL
- link leg_r4_link: geometry collision box size=0.08 0.08 0.32; visual mesh filename=package://atom_urdf/meshes/leg_r4_link.STL
- link leg_r5_link: geometry visual mesh filename=package://atom_urdf/meshes/leg_r5_link.STL
- link leg_r6_link: geometry collision box size=0.25 0.1 0.02; visual mesh filename=package://atom_urdf/meshes/leg_r6_link.STL
- link pelvis: geometry visual mesh filename=package://atom_urdf/meshes/pelvis.STL
- link right_elbow_roll_link: geometry visual mesh filename=package://atom_urdf/meshes/right_elbow_roll_link.STL
- link right_shoulder_roll_link: geometry collision box size=0.06 0.06 0.24; visual mesh filename=package://atom_urdf/meshes/right_shoulder_roll_link.STL
- link right_shoulder_yaw_link: geometry visual mesh filename=package://atom_urdf/meshes/right_shoulder_yaw_link.STL
- link right_wrist_pitch_link: geometry visual mesh filename=package://atom_urdf/meshes/right_wrist_pitch_link.STL
- link right_wrist_yaw_link: geometry visual mesh filename=package://atom_urdf/meshes/right_wrist_yaw_link.STL
- link torso_link: geometry collision box size=0.26 0.24 0.4; visual mesh filename=package://atom_urdf/meshes/torso_link.STL
Joints:
- removed joint uidx_l_arm_joint1
- removed joint uidx_l_arm_joint2
- removed joint uidx_r_arm_joint1
- removed joint uidx_r_arm_joint2
- added joint left_elbow_pitch_joint: type revolute, parent left_shoulder_yaw_link, child left_elbow_pitch_link, origin xyz=0.00044198773719138 0 -0.130000000000198 rpy=0 0 0, axis 0 1 0, limit lower=-1.57 upper=2 effort=36 velocity=2.62
- added joint left_shoulder_pitch_joint: type revolute, parent torso_link, child left_shoulder_pitch_link, origin xyz=0 0.128 0.333 rpy=0 0 0, axis 0 1 0, limit lower=-2.97 upper=2.97 effort=56 velocity=2.62
- added joint right_elbow_pitch_joint: type revolute, parent right_shoulder_yaw_link, child right_elbow_pitch_link, origin xyz=0.000441987737191488 0 -0.130000000000198 rpy=0 0 0, axis 0 1 0, limit lower=-1.57 upper=2 effort=36 velocity=2.62
- added joint right_shoulder_pitch_joint: type revolute, parent torso_link, child right_shoulder_pitch_link, origin xyz=0 -0.128 0.333 rpy=0 0 0, axis 0 1 0, limit lower=-2.97 upper=2.97 effort=56 velocity=2.62
- joint head_pitch_joint: type fixed -> revolute
- joint head_yaw_joint: type fixed -> revolute
- joint left_elbow_roll_joint: parent uidx_arm_l2_link -> left_elbow_pitch_link; type fixed -> revolute
- joint left_shoulder_roll_joint: parent uidx_arm_l1_link -> left_shoulder_pitch_link; type fixed -> revolute
- joint left_shoulder_yaw_joint: type fixed -> revolute
- joint left_wrist_pitch_joint: type fixed -> revolute
- joint left_wrist_yaw_joint: type fixed -> revolute
- joint right_elbow_roll_joint: parent uidx_arm_r2_link -> right_elbow_pitch_link; type fixed -> revolute
- joint right_shoulder_roll_joint: parent uidx_arm_r1_link -> right_shoulder_pitch_link; type fixed -> revolute
- joint right_shoulder_yaw_joint: type fixed -> revolute
- joint right_wrist_pitch_joint: type fixed -> revolute
- joint right_wrist_yaw_joint: type fixed -> revolute

File: urdf/atom_wholebody.urdf (robot description, URDF)
Before this commit: robot atom, 32 links, 31 joints
Links:
- removed link uidx_arm_l1_link
- removed link uidx_arm_l2_link
- removed link uidx_arm_r1_link
- removed link uidx_arm_r2_link
- added link left_elbow_pitch_link, mass 0.8548; collision box size=0.30 0.06 0.06; visual mesh filename=package://atom_urdf/meshes/left_elbow_pitch_link.STL
- added link left_shoulder_pitch_link, mass 0.4473; visual mesh filename=package://atom_urdf/meshes/left_shoulder_pitch_link.STL
- added link right_elbow_pitch_link, mass 0.8548; collision box size=0.30 0.06 0.06; visual mesh filename=package://atom_urdf/meshes/right_elbow_pitch_link.STL
- added link right_shoulder_pitch_link, mass 0.4473; visual mesh filename=package://atom_urdf/meshes/right_shoulder_pitch_link.STL
- link head_pitch_link: geometry collision box size=0.16 0.14 0.14; visual mesh filename=package://atom_urdf/meshes/head_pitch_link.STL
- link head_yaw_link: geometry visual mesh filename=package://atom_urdf/meshes/head_yaw_link.STL
- link left_elbow_roll_link: geometry visual mesh filename=package://atom_urdf/meshes/left_elbow_roll_link.STL
- link left_shoulder_roll_link: geometry collision box size=0.06 0.06 0.24; visual mesh filename=package://atom_urdf/meshes/left_shoulder_roll_link.STL
- link left_shoulder_yaw_link: geometry visual mesh filename=package://atom_urdf/meshes/left_shoulder_yaw_link.STL
- link left_wrist_pitch_link: geometry visual mesh filename=package://atom_urdf/meshes/left_wrist_pitch_link.STL
- link left_wrist_yaw_link: geometry visual mesh filename=package://atom_urdf/meshes/left_wrist_yaw_link.STL
- link leg_l1_link: geometry visual mesh filename=package://atom_urdf/meshes/leg_l1_link.STL
- link leg_l2_link: geometry visual mesh filename=package://atom_urdf/meshes/leg_l2_link.STL
- link leg_l3_link: geometry collision box size=0.08 0.08 0.24; visual mesh filename=package://atom_urdf/meshes/leg_l3_link.STL
- link leg_l4_link: geometry collision box size=0.08 0.08 0.32; visual mesh filename=package://atom_urdf/meshes/leg_l4_link.STL
- link leg_l5_link: geometry visual mesh filename=package://atom_urdf/meshes/leg_l5_link.STL
- link leg_l6_link: geometry collision box size=0.25 0.1 0.02; visual mesh filename=package://atom_urdf/meshes/leg_l6_link.STL
- link leg_r1_link: geometry visual mesh filename=package://atom_urdf/meshes/leg_r1_link.STL
- link leg_r2_link: geometry visual mesh filename=package://atom_urdf/meshes/leg_r2_link.STL
- link leg_r3_link: geometry collision box size=0.08 0.08 0.24; visual mesh filename=package://atom_urdf/meshes/leg_r3_link.STL
- link leg_r4_link: geometry collision box size=0.08 0.08 0.32; visual mesh filename=package://atom_urdf/meshes/leg_r4_link.STL
- link leg_r5_link: geometry visual mesh filename=package://atom_urdf/meshes/leg_r5_link.STL
- link leg_r6_link: geometry collision box size=0.25 0.1 0.02; visual mesh filename=package://atom_urdf/meshes/leg_r6_link.STL
- link pelvis: geometry visual mesh filename=package://atom_urdf/meshes/pelvis.STL
- link right_elbow_roll_link: geometry visual mesh filename=package://atom_urdf/meshes/right_elbow_roll_link.STL
- link right_shoulder_roll_link: geometry collision box size=0.06 0.06 0.24; visual mesh filename=package://atom_urdf/meshes/right_shoulder_roll_link.STL
- link right_shoulder_yaw_link: geometry visual mesh filename=package://atom_urdf/meshes/right_shoulder_yaw_link.STL
- link right_wrist_pitch_link: geometry visual mesh filename=package://atom_urdf/meshes/right_wrist_pitch_link.STL
- link right_wrist_yaw_link: geometry visual mesh filename=package://atom_urdf/meshes/right_wrist_yaw_link.STL
- link torso_link: geometry collision box size=0.26 0.24 0.4; visual mesh filename=package://atom_urdf/meshes/torso_link.STL
Joints:
- removed joint uidx_l_arm_joint1
- removed joint uidx_l_arm_joint2
- removed joint uidx_r_arm_joint1
- removed joint uidx_r_arm_joint2
- added joint left_elbow_pitch_joint: type revolute, parent left_shoulder_yaw_link, child left_elbow_pitch_link, origin xyz=0.00044198773719138 0 -0.130000000000198 rpy=0 0 0, axis 0 1 0, limit lower=-1.57 upper=2 effort=36 velocity=2.62
- added joint left_shoulder_pitch_joint: type revolute, parent torso_link, child left_shoulder_pitch_link, origin xyz=0 0.128 0.333 rpy=0 0 0, axis 0 1 0, limit lower=-2.97 upper=2.97 effort=56 velocity=2.62
- added joint right_elbow_pitch_joint: type revolute, parent right_shoulder_yaw_link, child right_elbow_pitch_link, origin xyz=0.000441987737191488 0 -0.130000000000198 rpy=0 0 0, axis 0 1 0, limit lower=-1.57 upper=2 effort=36 velocity=2.62
- added joint right_shoulder_pitch_joint: type revolute, parent torso_link, child right_shoulder_pitch_link, origin xyz=0 -0.128 0.333 rpy=0 0 0, axis 0 1 0, limit lower=-2.97 upper=2.97 effort=56 velocity=2.62
- joint left_elbow_roll_joint: parent uidx_arm_l2_link -> left_elbow_pitch_link
- joint left_shoulder_roll_joint: parent uidx_arm_l1_link -> left_shoulder_pitch_link
- joint right_elbow_roll_joint: parent uidx_arm_r2_link -> right_elbow_pitch_link
- joint right_shoulder_roll_joint: parent uidx_arm_r1_link -> right_shoulder_pitch_link
