Commit message: feat: p3-urdf

File: atom-p2/urdf/atom.urdf (robot description, URDF)
Before this commit: robot atom, 32 links, 31 joints
Links:
- removed link world
- link head_pitch_link: geometry collision box size=0.16 0.14 0.14; visual mesh filename=package://atom_p2/meshes/head_pitch_link.STL
- link head_yaw_link: geometry visual mesh filename=package://atom_p2/meshes/head_yaw_link.STL
- link left_elbow_pitch_link: geometry collision box size=0.30 0.06 0.06; visual mesh filename=package://atom_p2/meshes/left_elbow_pitch_link.STL
- link left_elbow_roll_link: geometry visual mesh filename=package://atom_p2/meshes/left_elbow_roll_link.STL
- link left_shoulder_pitch_link: geometry visual mesh filename=package://atom_p2/meshes/left_shoulder_pitch_link.STL
- link left_shoulder_roll_link: geometry collision box size=0.06 0.06 0.24; visual mesh filename=package://atom_p2/meshes/left_shoulder_roll_link.STL
- link left_shoulder_yaw_link: geometry visual mesh filename=package://atom_p2/meshes/left_shoulder_yaw_link.STL
- link left_wrist_pitch_link: geometry visual mesh filename=package://atom_p2/meshes/left_wrist_pitch_link.STL
- link left_wrist_yaw_link: geometry visual mesh filename=package://atom_p2/meshes/left_wrist_yaw_link.STL
- link leg_l1_link: geometry visual mesh filename=package://atom_p2/meshes/leg_l1_link.STL
- link leg_l2_link: geometry visual mesh filename=package://atom_p2/meshes/leg_l2_link.STL
- link leg_l3_link: geometry collision box size=0.08 0.08 0.24; visual mesh filename=package://atom_p2/meshes/leg_l3_link.STL
- link leg_l4_link: geometry collision box size=0.08 0.08 0.32; visual mesh filename=package://atom_p2/meshes/leg_l4_link.STL
- link leg_l5_link: geometry visual mesh filename=package://atom_p2/meshes/leg_l5_link.STL
- link leg_l6_link: geometry collision box size=0.25 0.1 0.02; visual mesh filename=package://atom_p2/meshes/leg_l6_link.STL
- link leg_r1_link: geometry visual mesh filename=package://atom_p2/meshes/leg_r1_link.STL
- link leg_r2_link: geometry visual mesh filename=package://atom_p2/meshes/leg_r2_link.STL
- link leg_r3_link: geometry collision box size=0.08 0.08 0.24; visual mesh filename=package://atom_p2/meshes/leg_r3_link.STL
- link leg_r4_link: geometry collision box size=0.08 0.08 0.32; visual mesh filename=package://atom_p2/meshes/leg_r4_link.STL
- link leg_r5_link: geometry visual mesh filename=package://atom_p2/meshes/leg_r5_link.STL
- link leg_r6_link: geometry collision box size=0.25 0.1 0.02; visual mesh filename=package://atom_p2/meshes/leg_r6_link.STL
- link pelvis: geometry visual mesh filename=package://atom_p2/meshes/pelvis.STL
- link right_elbow_pitch_link: geometry collision box size=0.30 0.06 0.06; visual mesh filename=package://atom_p2/meshes/right_elbow_pitch_link.STL
- link right_elbow_roll_link: geometry visual mesh filename=package://atom_p2/meshes/right_elbow_roll_link.STL
- link right_shoulder_pitch_link: geometry visual mesh filename=package://atom_p2/meshes/right_shoulder_pitch_link.STL
- link right_shoulder_roll_link: geometry collision box size=0.06 0.06 0.24; visual mesh filename=package://atom_p2/meshes/right_shoulder_roll_link.STL
- link right_shoulder_yaw_link: geometry visual mesh filename=package://atom_p2/meshes/right_shoulder_yaw_link.STL
- link right_wrist_pitch_link: geometry visual mesh filename=package://atom_p2/meshes/right_wrist_pitch_link.STL
- link right_wrist_yaw_link: geometry visual mesh filename=package://atom_p2/meshes/right_wrist_yaw_link.STL
- link torso_link: geometry collision box size=0.26 0.24 0.4; visual mesh filename=package://atom_p2/meshes/torso_link.STL
Joints:
- removed joint floating_base_joint
- joint torso_joint: type fixed -> revolute

File: atom-p2/urdf/atom_lower.urdf (robot description, URDF)
Before this commit: robot atom, 31 links, 30 joints
Links:
- added link world
- link head_pitch_link: geometry collision box size=0.16 0.14 0.14; visual mesh filename=package://atom_p2/meshes/head_pitch_link.STL
- link head_yaw_link: geometry visual mesh filename=package://atom_p2/meshes/head_yaw_link.STL
- link left_elbow_pitch_link: geometry collision box size=0.30 0.06 0.06; visual mesh filename=package://atom_p2/meshes/left_elbow_pitch_link.STL
- link left_elbow_roll_link: geometry visual mesh filename=package://atom_p2/meshes/left_elbow_roll_link.STL
- link left_shoulder_pitch_link: geometry visual mesh filename=package://atom_p2/meshes/left_shoulder_pitch_link.STL
- link left_shoulder_roll_link: geometry collision box size=0.06 0.06 0.24; visual mesh filename=package://atom_p2/meshes/left_shoulder_roll_link.STL
- link left_shoulder_yaw_link: geometry visual mesh filename=package://atom_p2/meshes/left_shoulder_yaw_link.STL
- link left_wrist_pitch_link: geometry visual mesh filename=package://atom_p2/meshes/left_wrist_pitch_link.STL
- link left_wrist_yaw_link: geometry visual mesh filename=package://atom_p2/meshes/left_wrist_yaw_link.STL
- link leg_l1_link: geometry visual mesh filename=package://atom_p2/meshes/leg_l1_link.STL
- link leg_l2_link: geometry visual mesh filename=package://atom_p2/meshes/leg_l2_link.STL
- link leg_l3_link: geometry collision box size=0.08 0.08 0.24; visual mesh filename=package://atom_p2/meshes/leg_l3_link.STL
- link leg_l4_link: geometry collision box size=0.08 0.08 0.32; visual mesh filename=package://atom_p2/meshes/leg_l4_link.STL
- link leg_l5_link: geometry visual mesh filename=package://atom_p2/meshes/leg_l5_link.STL
- link leg_l6_link: geometry collision box size=0.25 0.1 0.02; visual mesh filename=package://atom_p2/meshes/leg_l6_link.STL
- link leg_r1_link: geometry visual mesh filename=package://atom_p2/meshes/leg_r1_link.STL
- link leg_r2_link: geometry visual mesh filename=package://atom_p2/meshes/leg_r2_link.STL
- link leg_r3_link: geometry collision box size=0.08 0.08 0.24; visual mesh filename=package://atom_p2/meshes/leg_r3_link.STL
- link leg_r4_link: geometry collision box size=0.08 0.08 0.32; visual mesh filename=package://atom_p2/meshes/leg_r4_link.STL
- link leg_r5_link: geometry visual mesh filename=package://atom_p2/meshes/leg_r5_link.STL
- link leg_r6_link: geometry collision box size=0.25 0.1 0.02; visual mesh filename=package://atom_p2/meshes/leg_r6_link.STL
- link pelvis: geometry visual mesh filename=package://atom_p2/meshes/pelvis.STL
- link right_elbow_pitch_link: geometry collision box size=0.30 0.06 0.06; visual mesh filename=package://atom_p2/meshes/right_elbow_pitch_link.STL
- link right_elbow_roll_link: geometry visual mesh filename=package://atom_p2/meshes/right_elbow_roll_link.STL
- link right_shoulder_pitch_link: geometry visual mesh filename=package://atom_p2/meshes/right_shoulder_pitch_link.STL
- link right_shoulder_roll_link: geometry collision box size=0.06 0.06 0.24; visual mesh filename=package://atom_p2/meshes/right_shoulder_roll_link.STL
- link right_shoulder_yaw_link: geometry visual mesh filename=package://atom_p2/meshes/right_shoulder_yaw_link.STL
- link right_wrist_pitch_link: geometry visual mesh filename=package://atom_p2/meshes/right_wrist_pitch_link.STL
- link right_wrist_yaw_link: geometry visual mesh filename=package://atom_p2/meshes/right_wrist_yaw_link.STL
- link torso_link: geometry collision box size=0.26 0.24 0.4; visual mesh filename=package://atom_p2/meshes/torso_link.STL
Joints:
- added joint floating_base_joint: type floating, parent world, child pelvis
- joint torso_joint: type revolute -> fixed

File: atom-p2/urdf/atom_wholebody.urdf (robot description, URDF)
Before this commit: robot atom, 32 links, 31 joints
Links:
- link head_pitch_link: geometry collision box size=0.16 0.14 0.14; visual mesh filename=package://atom_p2/meshes/head_pitch_link.STL
- link head_yaw_link: geometry visual mesh filename=package://atom_p2/meshes/head_yaw_link.STL
- link left_elbow_pitch_link: geometry collision box size=0.30 0.06 0.06; visual mesh filename=package://atom_p2/meshes/left_elbow_pitch_link.STL
- link left_elbow_roll_link: geometry visual mesh filename=package://atom_p2/meshes/left_elbow_roll_link.STL
- link left_shoulder_pitch_link: geometry visual mesh filename=package://atom_p2/meshes/left_shoulder_pitch_link.STL
- link left_shoulder_roll_link: geometry collision box size=0.06 0.06 0.24; visual mesh filename=package://atom_p2/meshes/left_shoulder_roll_link.STL
- link left_shoulder_yaw_link: geometry visual mesh filename=package://atom_p2/meshes/left_shoulder_yaw_link.STL
- link left_wrist_pitch_link: geometry visual mesh filename=package://atom_p2/meshes/left_wrist_pitch_link.STL
- link left_wrist_yaw_link: geometry visual mesh filename=package://atom_p2/meshes/left_wrist_yaw_link.STL
- link leg_l1_link: geometry visual mesh filename=package://atom_p2/meshes/leg_l1_link.STL
- link leg_l2_link: geometry visual mesh filename=package://atom_p2/meshes/leg_l2_link.STL
- link leg_l3_link: geometry collision box size=0.08 0.08 0.24; visual mesh filename=package://atom_p2/meshes/leg_l3_link.STL
- link leg_l4_link: geometry collision box size=0.08 0.08 0.32; visual mesh filename=package://atom_p2/meshes/leg_l4_link.STL
- link leg_l5_link: geometry visual mesh filename=package://atom_p2/meshes/leg_l5_link.STL
- link leg_l6_link: geometry collision box size=0.25 0.1 0.02; visual mesh filename=package://atom_p2/meshes/leg_l6_link.STL
- link leg_r1_link: geometry visual mesh filename=package://atom_p2/meshes/leg_r1_link.STL
- link leg_r2_link: geometry visual mesh filename=package://atom_p2/meshes/leg_r2_link.STL
- link leg_r3_link: geometry collision box size=0.08 0.08 0.24; visual mesh filename=package://atom_p2/meshes/leg_r3_link.STL
- link leg_r4_link: geometry collision box size=0.08 0.08 0.32; visual mesh filename=package://atom_p2/meshes/leg_r4_link.STL
- link leg_r5_link: geometry visual mesh filename=package://atom_p2/meshes/leg_r5_link.STL
- link leg_r6_link: geometry collision box size=0.25 0.1 0.02; visual mesh filename=package://atom_p2/meshes/leg_r6_link.STL
- link pelvis: geometry visual mesh filename=package://atom_p2/meshes/pelvis.STL
- link right_elbow_pitch_link: geometry collision box size=0.30 0.06 0.06; visual mesh filename=package://atom_p2/meshes/right_elbow_pitch_link.STL
- link right_elbow_roll_link: geometry visual mesh filename=package://atom_p2/meshes/right_elbow_roll_link.STL
- link right_shoulder_pitch_link: geometry visual mesh filename=package://atom_p2/meshes/right_shoulder_pitch_link.STL
- link right_shoulder_roll_link: geometry collision box size=0.06 0.06 0.24; visual mesh filename=package://atom_p2/meshes/right_shoulder_roll_link.STL
- link right_shoulder_yaw_link: geometry visual mesh filename=package://atom_p2/meshes/right_shoulder_yaw_link.STL
- link right_wrist_pitch_link: geometry visual mesh filename=package://atom_p2/meshes/right_wrist_pitch_link.STL
- link right_wrist_yaw_link: geometry visual mesh filename=package://atom_p2/meshes/right_wrist_yaw_link.STL
- link torso_link: geometry collision box size=0.26 0.24 0.4; visual mesh filename=package://atom_p2/meshes/torso_link.STL
